File: HARDWARE/JACK-BOARD/KOSMO-POLY6-JACKS.kicad_pcb (KiCad board)
At the start: 2 copper layers, 70 x 175 mm, 30 parts, among them J1 RAMP_OUT0, J10 RAMP_OUT3, J11 PULSE_OUT3, J12 GATE_OUT3, J13 RAMP_OUT4, J14 PULSE_OUT4, J15 GATE_OUT4, J16 RAMP_OUT5, J17 PULSE_OUT5, J18 GATE_OUT5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

Commit message: sync
Routing:
- net GND-S: track 0.00 -> 577.3 mm
- net GATE_OUT2-S: track 0.00 -> 171.5 mm
- net GATE_OUT1-S: track 0.00 -> 151.3 mm
- net RAMP_OUT5-S: track 0.00 -> 148.4 mm
- net PULSE_OUT5-S: track 0.00 -> 143.4 mm
- net PULSE_OUT5-N: track 0.00 -> 140.8 mm
- net GATE_OUT2-N: track 0.00 -> 138.6 mm
- net GATE_OUT3-S: track 0.00 -> 136.4 mm
- net RAMP_OUT5-N: track 0.00 -> 135.8 mm
- net RAMP_OUT4-S: track 0.00 -> 127.6 mm
- net PULSE_OUT4-S: track 0.00 -> 123.3 mm
- net PULSE_OUT4-N: track 0.00 -> 120.3 mm
- net GATE_OUT1-N: track 0.00 -> 119.4 mm
- net RAMP_OUT4-N: track 0.00 -> 115.4 mm
- net RAMP_OUT3-S: track 0.00 -> 105.4 mm
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- removed copper zone on B.Cu, net GND-S

Commit message: Kicad7 and Fixlayered
Other:
- net class Default removed

Commit message: holidaysync
Parts:
- J1, J10, J11, J12, J13, J14, J15, J16, J17, J18, J2, J3, J4, J5, J6, J7, J8, J9: footprint AA-ROB-FULL:Jack_6.5mmLMNC -> JACK-BOARD:Jack_6.5mmLMNC
Connections:
- GATE_IN1 pad 4: GATE_OUT1-S -> GATE_OUT4-S
- GATE_IN1 pad 6: GATE_OUT2-S -> GATE_OUT5-S
- GATE_OUT1 pad 4: GATE_OUT1-N -> GATE_OUT4-N
- GATE_OUT1 pad 6: GATE_OUT2-N -> GATE_OUT5-N
- H1 pad 1: GND-S -> Net-(H1-Pad1)
- H2 pad 1: GND-S -> Net-(H1-Pad1)
- H3 pad 1: GND-S -> Net-(H1-Pad1)
- H4 pad 1: GND-S -> Net-(H1-Pad1)
- J1 pad S: Net-(J1-PadS) -> unconnected-(J1-PadS)
- J1 pad SN: Net-(J1-PadSN) -> unconnected-(J1-PadSN)
- J10 pad S: Net-(J10-PadS) -> unconnected-(J10-PadS)
- J10 pad SN: Net-(J10-PadSN) -> unconnected-(J10-PadSN)
- J11 pad S: Net-(J11-PadS) -> unconnected-(J11-PadS)
- J11 pad SN: Net-(J11-PadSN) -> unconnected-(J11-PadSN)
- J12 pad S: Net-(J12-PadS) -> unconnected-(J12-PadS)
- J12 pad SN: Net-(J12-PadSN) -> unconnected-(J12-PadSN)
- J13 pad S: Net-(J13-PadS) -> unconnected-(J13-PadS)
- J13 pad SN: Net-(J13-PadSN) -> unconnected-(J13-PadSN)
- J14 pad S: Net-(J14-PadS) -> unconnected-(J14-PadS)
- J14 pad SN: Net-(J14-PadSN) -> unconnected-(J14-PadSN)
- J15 pad S: Net-(J15-PadS) -> unconnected-(J15-PadS)
- J15 pad SN: Net-(J15-PadSN) -> unconnected-(J15-PadSN)
- J15 pad T: GATE_OUT1-S -> GATE_OUT4-S
- J15 pad TN: GATE_OUT1-N -> GATE_OUT4-N
- J16 pad S: Net-(J16-PadS) -> unconnected-(J16-PadS)
- J16 pad SN: Net-(J16-PadSN) -> unconnected-(J16-PadSN)
- J17 pad S: Net-(J17-PadS) -> unconnected-(J17-PadS)
- J17 pad SN: Net-(J17-PadSN) -> unconnected-(J17-PadSN)
- J18 pad S: Net-(J18-PadS) -> unconnected-(J18-PadS)
- J18 pad SN: Net-(J18-PadSN) -> unconnected-(J18-PadSN)
- J18 pad T: GATE_OUT2-S -> GATE_OUT5-S
- J18 pad TN: GATE_OUT2-N -> GATE_OUT5-N
- J2 pad S: Net-(J2-PadS) -> unconnected-(J2-PadS)
- J2 pad SN: Net-(J2-PadSN) -> unconnected-(J2-PadSN)
- J3 pad S: Net-(J3-PadS) -> unconnected-(J3-PadS)
- J3 pad SN: Net-(J3-PadSN) -> unconnected-(J3-PadSN)
- J4 pad S: Net-(J4-PadS) -> unconnected-(J4-PadS)
- J4 pad SN: Net-(J4-PadSN) -> unconnected-(J4-PadSN)
- J5 pad S: Net-(J5-PadS) -> unconnected-(J5-PadS)
- J5 pad SN: Net-(J5-PadSN) -> unconnected-(J5-PadSN)
- J6 pad S: Net-(J6-PadS) -> unconnected-(J6-PadS)
- J6 pad SN: Net-(J6-PadSN) -> unconnected-(J6-PadSN)
- J7 pad S: Net-(J7-PadS) -> unconnected-(J7-PadS)
- J7 pad SN: Net-(J7-PadSN) -> unconnected-(J7-PadSN)
- J8 pad S: Net-(J8-PadS) -> unconnected-(J8-PadS)
- J8 pad SN: Net-(J8-PadSN) -> unconnected-(J8-PadSN)
- J9 pad S: Net-(J9-PadS) -> unconnected-(J9-PadS)
- J9 pad SN: Net-(J9-PadSN) -> unconnected-(J9-PadSN)
Routing:
- net Net-(H1-Pad1): track 0.00 -> 293.4 mm
- net GATE_OUT5-S: track 0.00 -> 152.1 mm
- net GATE_OUT5-N: track 0.00 -> 134.2 mm
- net GATE_OUT4-S: track 0.00 -> 132.6 mm
- net GATE_OUT4-N: track 0.00 -> 114.3 mm
- net GATE_OUT2-S: track 171.5 -> 79.9 mm
- net GATE_OUT1-S: track 151.3 -> 60.7 mm
- net GND-S: track 577.3 -> 495.2 mm
- net GATE_OUT1-N: track 119.4 -> 43.9 mm
- net GATE_OUT2-N: track 138.6 -> 73.2 mm
- net PULSE_OUT5-N: track 140.8 -> 168.7 mm
- net GATE_OUT3-S: track 136.4 -> 111.0 mm
- net PULSE_OUT4-N: track 120.3 -> 145.7 mm
- net PULSE_OUT3-N: track 99.9 -> 122.4 mm
- net PULSE_OUT1-N: track 62.2 -> 80.3 mm
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- added copper zone on B.Cu, net GND-S
